File: PCB/Drone Lights/Drone Lights.kicad_pcb (KiCad board)
At the start: 2 copper layers, 25.4 x 74.5 mm, 37 parts, among them J1 Proto Pin, J10 Prog_Connector, J11 Proto Pin, J12 Proto Pin, J13 Proto Pin, J14 Proto Pin, J2 Input, J3 Proto Pin, J4 Proto Pin, J5 Proto Pin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

Commit message: Updated with local copy
Parts:
- D1: value LED -> LED 2.85V 350 mA
- R1: value 10 -> 10 1.25W
Connections:
- net PROG_MISO renamed MOSI
- net PROG_MOSI renamed MISO
